File: PCB/Controller.sch (KiCad schematic (older format))
At the start: 12 parts, among them IC501 ATMEGA88-A, P501 PRG, SW501 Time Set, SW502 Alarm Set, SW503 Fast, SW504 Slow, SW505 Auto Time, SW506 Sleep, SW507 Sleep, SW508 Alarm Enabled

Commit message: Added the tactile switch
Parts:
- removed SW501: Time Set, symbol SW_PUSH
- removed SW502: Alarm Set, symbol SW_PUSH
- removed SW503: Fast, symbol SW_PUSH
- removed SW504: Slow, symbol SW_PUSH
- removed SW506: Sleep, symbol SW_PUSH
- added SW501: Time Set, tfac-footprints:TL3315, symbol TL3315NF160Q
- added SW502: Alarm Set, tfac-footprints:TL3315, symbol TL3315NF160Q
- added SW503: Fast, tfac-footprints:TL3315, symbol TL3315NF160Q
- added SW504: Slow, tfac-footprints:TL3315, symbol TL3315NF160Q
- added SW506: Sleep, tfac-footprints:TL3315, symbol TL3315NF160Q
- SW507: value Sleep -> Summer Time
Connections:
- no-connect marks 9 -> 19
Other:
- moved on the sheet: SW505
Changed lines of the file:
@@
 Reset
-$Comp
-L SW_PUSH SW501
-U 1 1 55C0F652
-P 9350 2450
-F 0 "SW501" H 9500 2560 50  0000 C CNN
-F 1 "Time Set" H 9350 2370 50  0000 C CNN
-F 2 "" H 9350 2450 60  0001 C CNN
-F 3 "" H 9350 2450 60  0000 C CNN
-	1    9350 2450
-	1    0    0    -1
-$EndComp
-$Comp
-L SW_PUSH SW502
-U 1 1 55C0F6D0
-P 9350 2750
-F 0 "SW502" H 9500 2860 50  0000 C CNN
-F 1 "Alarm Set" H 9350 2670 50  0000 C CNN
-F 2 "" H 9350 2750 60  0001 C CNN
-F 3 "" H 9350 2750 60  0000 C CNN
-	1    9350 2750
-	1    0    0    -1
-$EndComp
-$Comp
-L SW_PUSH SW503
-U 1 1 55C0F704
-P 9350 3050
-F 0 "SW503" H 9500 3160 50  0000 C CNN
-F 1 "Fast" H 9350 2970 50  0000 C CNN
-F 2 "" H 9350 3050 60  0001 C CNN
-F 3 "" H 9350 3050 60  0000 C CNN
-	1    9350 3050
-	1    0    0    -1
-$EndComp
-$Comp
-L SW_PUSH SW504
-U 1 1 55C0F741
-P 9350 3350
-F 0 "SW504" H 9500 3460 50  0000 C CNN
-F 1 "Slow" H 9350 3270 50  0000 C CNN
-F 2 "" H 9350 3350 60  0001 C CNN
-F 3 "" H 9350 3350 60  0000 C CNN
-	1    9350 3350
-	1    0    0    -1
-$EndComp
 $Comp
 L SW_PUSH SW505
 U 1 1 55C0F785
-P 9350 3650
-F 0 "SW505" H 9500 3760 50  0000 C CNN
-F 1 "Auto Time" H 9350 3570 50  0000 C CNN
-F 2 "" H 9350 3650 60  0001 C CNN
-F 3 "" H 9350 3650 60  0000 C CNN
-	1    9350 3650
-	1    0    0    -1
-$EndComp
-$Comp
-L SW_PUSH SW506
-U 1 1 55C0F89E
-P 9350 4000
-F 0 "SW506" H 9500 4110 50  0000 C CNN
-F 1 "Sleep" H 9350 3920 50  0000 C CNN
-F 2 "" H 9350 4000 60  0001 C CNN
-F 3 "" H 9350 4000 60  0000 C CNN
-	1    9350 4000
+P 9350 3500
+F 0 "SW505" H 9500 3610 50  0000 C CNN
+F 1 "Auto Time" H 9350 3420 50  0000 C CNN
+F 2 "" H 9350 3500 60  0001 C CNN
+F 3 "" H 9350 3500 60  0000 C CNN
+	1    9350 3500
 	1    0    0    -1
 $EndComp
@@
 U 1 1 55C0F8D0
 P 9400 4800
-F 0 "SW508" H 9400 4900 50  0000 C CNN
+F 0 "SW508" H 9150 4950 50  0000 C CNN
 F 1 "Alarm Enabled" H 9400 4700 50  0000 C CNN
 F 2 "" H 9400 4800 60  0001 C CNN
@@
 	1    0    0    -1
 $EndComp
-Text GLabel 8700 2450 0    60   Input ~ 0
+Text GLabel 8700 1850 0    60   Input ~ 0
 Time_Set
+Text GLabel 8700 2300 0    60   Input ~ 0
+Alarm_Set
 Text GLabel 8700 2750 0    60   Input ~ 0
-Alarm_Set
-Text GLabel 8700 3050 0    60   Input ~ 0
 Fast
-Text GLabel 8700 3350 0    60   Input ~ 0
+Text GLabel 8700 3200 0    60   Input ~ 0
 Slow
-Text GLabel 8700 3650 0    60   Input ~ 0
+Text GLabel 8700 3500 0    60   Input ~ 0
 Auto_Time
 Text GLabel 8700 4000 0    60   Input ~ 0
@@
 U 1 1 55C107C5
 P 9350 4350
-F 0 "SW507" H 9500 4460 50  0000 C CNN
-F 1 "Sleep" H 9350 4270 50  0000 C CNN
+F 0 "SW507" H 9000 4450 50  0000 C CNN
+F 1 "Summer Time" H 9350 4270 50  0000 C CNN
 F 2 "" H 9350 4350 60  0001 C CNN
 F 3 "" H 9350 4350 60  0000 C CNN
@@
 Connection ~ 2900 2200
 Wire Wire Line
-	9650 2450 10100 2450
-Wire Wire Line
-	10100 2450 10100 5000
-Wire Wire Line
-	9650 2750 10100 2750
+	10100 1850 10100 5000
+Wire Wire Line
+	9550 2750 10100 2750
 Connection ~ 10100 2750
 Wire Wire Line
-	9650 3050 10100 3050
-Connection ~ 10100 3050
-Wire Wire Line
-	9650 3350 10100 3350
-Connection ~ 10100 3350
-Wire Wire Line
-	9650 3650 10100 3650
-Connection ~ 10100 3650
-Wire Wire Line
-	9650 4000 10100 4000
+	9550 3200 10100 3200
+Connection ~ 10100 3200
+Wire Wire Line
+	9650 3500 10100 3500
+Connection ~ 10100 3500
+Wire Wire Line
+	9550 4000 10100 4000
 Connection ~ 10100 4000
 Wire Wire Line
-	8700 2450 9050 2450
+	8700 1850 9050 1850
+Wire Wire Line
+	8700 2300 9050 2300
 Wire Wire Line
 	8700 2750 9050 2750
 Wire Wire Line
-	8700 3050 9050 3050
-Wire Wire Line
-	8700 3350 9050 3350
-Wire Wire Line
-	8700 3650 9050 3650
+	8700 3200 9050 3200
+Wire Wire Line
+	8700 3500 9050 3500
 Wire Wire Line
 	8700 4000 9050 4000
@@
 Connection ~ 10100 4350
 Wire Wire Line
-	9900 4800 10100 4800
+	10100 4800 9900 4800
 Connection ~ 10100 4800
 Text GLabel 5900 4400 2    60   Input ~ 0
@@
 NoConn ~ 3750 3550
 NoConn ~ 3750 2800
+$Comp
+L TL3315NF160Q SW501
+U 1 1 55D05D88
+P 9300 1750
+F 0 "SW501" V 9300 2100 60  0000 C CNN
+F 1 "Time Set" V 9150 1750 60  0000 C CNN
+F 2 "tfac-footprints:TL3315" H 9300 1700 60  0001 C CNN
+F 3 "" H 9300 1700 60  0000 C CNN
+F 4 "Value" H 9300 1750 60  0001 C CNN "MPN"
+F 5 "Value" H 9300 1750 60  0001 C CNN "ConradPN"
+F 6 "Value" H 9600 1750 60  0001 C CNN "Label"
+	1    9300 1750
+	0    -1   -1   0
+$EndComp
+Wire Wire Line
+	9550 1850 10100 1850
+$Comp
+L TL3315NF160Q SW502
+U 1 1 55D05FEA
+P 9300 2200
+F 0 "SW502" V 9300 2550 60  0000 C CNN
+F 1 "Alarm Set" V 9150 2200 60  0000 C CNN
+F 2 "tfac-footprints:TL3315" H 9300 2150 60  0001 C CNN
+F 3 "" H 9300 2150 60  0000 C CNN
+	1    9300 2200
+	0    -1   -1   0
+$EndComp
+Wire Wire Line
+	9550 2300 10100 2300
+Connection ~ 10100 2300
+$Comp
+L TL3315NF160Q SW503
+U 1 1 55D0627F
+P 9300 2650
+F 0 "SW503" V 9300 3000 60  0000 C CNN
+F 1 "Fast" V 9150 2650 60  0000 C CNN
+F 2 "tfac-footprints:TL3315" H 9300 2600 60  0001 C CNN
+F 3 "" H 9300 2600 60  0000 C CNN
+	1    9300 2650
+	0    -1   -1   0
+$EndComp
+$Comp
+L TL3315NF160Q SW504
+U 1 1 55D06309
+P 9300 3100
+F 0 "SW504" V 9300 3500 60  0000 C CNN
+F 1 "Slow" V 9150 3100 60  0000 C CNN
+F 2 "tfac-footprints:TL3315" H 9300 3050 60  0001 C CNN
+F 3 "" H 9300 3050 60  0000 C CNN
+	1    9300 3100
+	0    -1   -1   0
+$EndComp
+$Comp
+L TL3315NF160Q SW506
+U 1 1 55D06511
+P 9300 3900
+F 0 "SW506" V 9300 4300 60  0000 C CNN
+F 1 "Sleep" V 9150 3900 60  0000 C CNN
+F 2 "tfac-footprints:TL3315" H 9300 3850 60  0001 C CNN
+F 3 "" H 9300 3850 60  0000 C CNN
+	1    9300 3900
+	0    -1   -1   0
+$EndComp
+NoConn ~ 9050 1650
+NoConn ~ 9550 1650
+NoConn ~ 9050 2100
+NoConn ~ 9550 2100
+NoConn ~ 9050 2550
+NoConn ~ 9550 2550
+NoConn ~ 9050 3000
+NoConn ~ 9550 3000
+NoConn ~ 9050 3800
+NoConn ~ 9550 3800
 $EndSCHEMATC

Commit message: Added the switch footprints and started the layout
Parts:
- removed SW505: Auto Time, symbol SW_PUSH
- removed SW508: Alarm Enabled, symbol SPST
- added SW505: Auto Time, tfac-footprints:AYZ0202AGRLC, symbol SWITCH_INV
- added SW508: Alarm Enabled, tfac-footprints:CLSB12C01, symbol SWITCH_INV
- SW507: footprint (none) -> Pin_Headers:Pin_Header_Straight_1x02
Connections:
- wire segments 54 -> 84
- no-connect marks 19 -> 12
Other:
- moved on the sheet: SW506, SW507

Commit message: Getting up to date
Connections:
- net Reset: now also IC501.18 (AVCC), IC501.4 (VCC), IC501.6 (VCC), R501.1; no longer IC501.29 ((PCINT14/~RESET~)PC6), R501.2
- new net: IC501.29 ((PCINT14/~RESET~)PC6), R501.2
Other:
- moved on the sheet: C501, R501
Changed lines of the file:
@@
 EESchema Schematic File Version 2
+LIBS:TfaC-rescue
 LIBS:power
 LIBS:device
@@
 L C C501
 U 1 1 5570FFE4
-P 2700 2500
-F 0 "C501" H 2725 2600 50  0000 L CNN
-F 1 "100n" H 2725 2400 50  0000 L CNN
-F 2 "Capacitors_SMD:C_0805_HandSoldering" H 2738 2350 30  0001 C CNN
-F 3 "" H 2700 2500 60  0000 C CNN
-	1    2700 2500
+P 3350 2500
+F 0 "C501" H 3375 2600 50  0000 L CNN
+F 1 "100n" H 3375 2400 50  0000 L CNN
+F 2 "Capacitors_SMD:C_0805_HandSoldering" H 3388 2350 30  0001 C CNN
+F 3 "" H 3350 2500 60  0000 C CNN
+	1    3350 2500
 	1    0    0    -1
 $EndComp
@@
 L GND #PWR011
 U 1 1 55710077
-P 2700 2900
-F 0 "#PWR011" H 2700 2650 50  0001 C CNN
-F 1 "GND" H 2700 2750 50  0000 C CNN
-F 2 "" H 2700 2900 60  0000 C CNN
-F 3 "" H 2700 2900 60  0000 C CNN
-	1    2700 2900
+P 3350 2900
+F 0 "#PWR011" H 3350 2650 50  0001 C CNN
+F 1 "GND" H 3350 2750 50  0000 C CNN
+F 2 "" H 3350 2900 60  0000 C CNN
+F 3 "" H 3350 2900 60  0000 C CNN
+	1    3350 2900
 	1    0    0    -1
 $EndComp
@@
 L R R501
 U 1 1 55710A4C
-P 3200 2200
-F 0 "R501" V 3280 2200 50  0000 C CNN
-F 1 "10K" V 3200 2200 50  0000 C CNN
-F 2 "Resistors_SMD:R_0805_HandSoldering" V 3130 2200 30  0001 C CNN
-F 3 "" H 3200 2200 30  0000 C CNN
-	1    3200 2200
+P 6550 3650
+F 0 "R501" V 6630 3650 50  0000 C CNN
+F 1 "10K" V 6550 3650 50  0000 C CNN
+F 2 "Resistors_SMD:R_0805_HandSoldering" V 6480 3650 30  0001 C CNN
+F 3 "" H 6550 3650 30  0000 C CNN
+	1    6550 3650
 	0    1    1    0
 $EndComp
 Text GLabel 6500 1400 0    60   Input ~ 0
 Reset
-Text GLabel 5900 3650 2    60   Input ~ 0
-Reset
-Text GLabel 3150 1700 2    60   Input ~ 0
+Text GLabel 3050 1950 0    60   Input ~ 0
 Reset
 $Comp
@@
 	7100 1300 6850 1300
 Wire Wire Line
-	2700 2650 2700 2900
-Wire Wire Line
-	2700 2350 2700 2200
-Wire Wire Line
-	3350 2200 3750 2200
+	3350 2650 3350 2900
 Connection ~ 3600 2200
 Wire Wire Line
-	2200 2200 3050 2200
-Connection ~ 2700 2200
-Wire Wire Line
 	6500 1400 7100 1400
-Wire Wire Line
-	5900 3650 5650 3650
-Wire Wire Line
-	3150 1700 2900 1700
-Wire Wire Line
-	2900 1700 2900 2200
-Connection ~ 2900 2200
 Wire Wire Line
 	10100 1750 10100 5850
@@
 NoConn ~ 9900 5450
 NoConn ~ 9300 3850
+Wire Wire Line
+	2200 2200 3750 2200
+Wire Wire Line
+	5650 3650 6400 3650
+Wire Wire Line
+	6700 3650 6900 3650
+Wire Wire Line
+	3350 2350 3350 2200
+Connection ~ 3350 2200
+Wire Wire Line
+	3050 1950 3200 1950
+Wire Wire Line
+	3200 1950 3200 2200
+Connection ~ 3200 2200
+Text HLabel 6900 3650 2    60   Input ~ 0
+Vcc
 $EndSCHEMATC
