File: PCB/powerSystem.sch (KiCad schematic (older format))
At the start: 0 parts

Commit message: Started the schematic. Added the power circuit
Parts:
- added C?: 100n, symbol C
- added C?: 4.7u, symbol C
- added P?: Vin, symbol CONN_01X01
- added P?: Vcc, symbol CONN_01X01
- added P?: GND, symbol CONN_01X01
- added P?: Vbb, symbol CONN_01X01
- added R?: 0, symbol R
- added R?: 3.3, symbol R
- added U?: MCP1703T-5002E/CB, symbol MCP1703T-5002E/CB
- added U?: LD2979, symbol LD2979
Connections:
- net labels added: GND, Vbb, Vcc, Vin
- wire segments 0 -> 24
Changed lines of the file:
@@
 LIBS:memory
 LIBS:xilinx
-LIBS:special
 LIBS:microcontrollers
 LIBS:dsp
@@
 LIBS:contrib
 LIBS:valves
+LIBS:Tfac-Symbols
+LIBS:TfaC-cache
 EELAYER 25 0
 EELAYER END
 $Descr A4 11693 8268
 encoding utf-8
-Sheet 1 5
+Sheet 2 5
 Title ""
 Date ""
@@
 Comment4 ""
 $EndDescr
+$Comp
+L MCP1703T-5002E/CB U?
+U 1 1 5565D3BF
+P 5000 2000
+F 0 "U?" H 5100 1850 50  0000 C CNN
+F 1 "MCP1703T-5002E/CB" H 5000 2150 50  0000 C CNN
+F 2 "" H 5000 2000 60  0000 C CNN
+F 3 "http://ww1.microchip.com/downloads/en/DeviceDoc/22049e.pdf" H 5000 2000 60  0001 C CNN
+F 4 "MCP1703T-5002E/CB" H 5000 2000 60  0001 C CNN "MPN"
+F 5 "651424 - 62" H 5000 2000 60  0001 C CNN "ConradPN"
+	1    5000 2000
+	1    0    0    -1
+$EndComp
+$Comp
+L GND #PWR?
+U 1 1 5565D42B
+P 5000 2600
+F 0 "#PWR?" H 5000 2350 50  0001 C CNN
+F 1 "GND" H 5000 2450 50  0000 C CNN
+F 2 "" H 5000 2600 60  0000 C CNN
+F 3 "" H 5000 2600 60  0000 C CNN
+	1    5000 2600
+	1    0    0    -1
+$EndComp
+Wire Wire Line
+	5000 2200 5000 2500
+Wire Wire Line
+	5000 2500 5000 2600
+Text HLabel 4050 2000 0    60   Input ~ 0
+Vin
+Wire Wire Line
+	4050 2000 4250 2000
+Wire Wire Line
+	4250 2000 4700 2000
+$Comp
+L CONN_01X01 P?
+U 1 1 5565D452
+P 4250 1600
+F 0 "P?" V 4250 1450 50  0000 C CNN
+F 1 "Vin" V 4350 1600 50  0000 C CNN
+F 2 "" H 4250 1600 60  0000 C CNN
+F 3 "" H 4250 1600 60  0000 C CNN
+	1    4250 1600
+	0    -1   -1   0
+$EndComp
+Connection ~ 4250 2000
+Wire Wire Line
+	5300 2000 5650 2000
+Wire Wire Line
+	5650 2000 5850 2000
+$Comp
+L CONN_01X01 P?
+U 1 1 5565D4A7
+P 5650 1600
+F 0 "P?" V 5650 1500 50  0000 C CNN
+F 1 "Vcc" V 5750 1600 50  0000 C CNN
+F 2 "" H 5650 1600 60  0000 C CNN
+F 3 "" H 5650 1600 60  0000 C CNN
+	1    5650 1600
+	0    -1   -1   0
+$EndComp
+Wire Wire Line
+	5650 1800 5650 2000
+Connection ~ 5650 2000
+$Comp
+L LD2979 U?
+U 1 1 5565DC6E
+P 5050 3450
+F 0 "U?" H 5250 3000 50  0000 C CNN
+F 1 "LD2979" H 5050 3600 50  0000 C CNN
+F 2 "" H 5050 3450 60  0000 C CNN
+F 3 "" H 5050 3450 60  0000 C CNN
+	1    5050 3450
+	1    0    0    -1
+$EndComp
+Wire Wire Line
+	4000 3450 4250 3450
+Wire Wire Line
+	4250 3450 4750 3450
+$Comp
+L C C?
+U 1 1 5565DCBC
+P 4250 3800
+F 0 "C?" H 4275 3900 50  0000 L CNN
+F 1 "100n" H 4275 3700 50  0000 L CNN
+F 2 "" H 4288 3650 30  0000 C CNN
+F 3 "" H 4250 3800 60  0000 C CNN
+	1    4250 3800
+	1    0    0    -1
+$EndComp
+$Comp
+L R R?
+U 1 1 5565DCEF
+P 4650 4150
+F 0 "R?" V 4730 4150 50  0000 C CNN
+F 1 "0" V 4650 4150 50  0000 C CNN
+F 2 "" V 4580 4150 30  0000 C CNN
+F 3 "" H 4650 4150 30  0000 C CNN
+	1    4650 4150
+	1    0    0    -1
+$EndComp
+Connection ~ 4250 3450
+$Comp
+L GND #PWR?
+U 1 1 5565DD5B
+P 4250 4600
+F 0 "#PWR?" H 4250 4350 50  0001 C CNN
+F 1 "GND" H 4250 4450 50  0000 C CNN
+F 2 "" H 4250 4600 60  0000 C CNN
+F 3 "" H 4250 4600 60  0000 C CNN
+	1    4250 4600
+	1    0    0    -1
+$EndComp
+Wire Wire Line
+	4250 3950 4250 4500
+Wire Wire Line
+	4250 4500 4250 4600
+Wire Wire Line
+	4750 3700 4650 3700
+Wire Wire Line
+	4650 3700 4650 4000
+Wire Wire Line
+	4650 4300 4650 4500
+Wire Wire Line
+	4650 4500 4250 4500
+Connection ~ 4250 4500
+Wire Wire Line
+	5350 3450 5650 3450
+Wire Wire Line
+	5650 3450 5900 3450
+$Comp
+L C C?
+U 1 1 5565DDF6
+P 5650 3800
+F 0 "C?" H 5675 3900 50  0000 L CNN
+F 1 "4.7u" H 5675 3700 50  0000 L CNN
+F 2 "" H 5688 3650 30  0000 C CNN
+F 3 "" H 5650 3800 60  0000 C CNN
+	1    5650 3800
+	1    0    0    -1
+$EndComp
+Wire Wire Line
+	5650 3300 5650 3450
+Wire Wire Line
+	5650 3450 5650 3650
+Connection ~ 5650 3450
+$Comp
+L R R?
+U 1 1 5565DE49
+P 5650 4300
+F 0 "R?" V 5730 4300 50  0000 C CNN
+F 1 "3.3" V 5650 4300 50  0000 C CNN
+F 2 "" V 5580 4300 30  0000 C CNN
+F 3 "" H 5650 4300 30  0000 C CNN
+	1    5650 4300
+	1    0    0    -1
+$EndComp
+Wire Wire Line
+	5650 3950 5650 4150
+$Comp
+L GND #PWR?
+U 1 1 5565DE90
+P 5650 4600
+F 0 "#PWR?" H 5650 4350 50  0001 C CNN
+F 1 "GND" H 5650 4450 50  0000 C CNN
+F 2 "" H 5650 4600 60  0000 C CNN
+F 3 "" H 5650 4600 60  0000 C CNN
+	1    5650 4600
+	1    0    0    -1
+$EndComp
+Wire Wire Line
+	5650 4450 5650 4600
+Text HLabel 5850 2000 2    60   Output ~ 0
+Vcc
+Text HLabel 5900 3450 2    60   Output ~ 0
+Vbb
+Wire Wire Line
+	4250 3450 4250 3650
+Text HLabel 4000 3450 0    60   Input ~ 0
+Vin
+Wire Wire Line
+	4250 1800 4250 2000
+$Comp
+L CONN_01X01 P?
+U 1 1 5565EA50
+P 4100 2500
+F 0 "P?" H 4100 2600 50  0000 C CNN
+F 1 "GND" H 4100 2400 50  0000 C CNN
+F 2 "" H 4100 2500 60  0000 C CNN
+F 3 "" H 4100 2500 60  0000 C CNN
+	1    4100 2500
+	-1   0    0    1
+$EndComp
+Wire Wire Line
+	4300 2500 5000 2500
+Connection ~ 5000 2500
+$Comp
+L CONN_01X01 P?
+U 1 1 5565EC08
+P 5650 3100
+F 0 "P?" V 5650 2950 50  0000 C CNN
+F 1 "Vbb" V 5750 3100 50  0000 C CNN
+F 2 "" H 5650 3100 60  0000 C CNN
+F 3 "" H 5650 3100 60  0000 C CNN
+	1    5650 3100
+	0    -1   -1   0
+$EndComp
 $EndSCHEMATC

Commit message: Corrected symbol for the LD2979 and filtering capacitors
Parts:
- removed R?: 0, symbol R
- removed R?: 3.3, symbol R
- removed U?: LD2979, symbol LD2979
- added C? (x2): 1u, symbol C
- added R?: 0, symbol R
- added U?: LD2979, symbol LD2979
- C?: value 100n -> 1u
- C?: value 4.7u -> 1u
Connections:
- wire segments 24 -> 29
Other:
- moved on the sheet: C?
Changed lines of the file:
@@
 L GND #PWR?
 U 1 1 5565D42B
-P 5000 2600
-F 0 "#PWR?" H 5000 2350 50  0001 C CNN
-F 1 "GND" H 5000 2450 50  0000 C CNN
-F 2 "" H 5000 2600 60  0000 C CNN
-F 3 "" H 5000 2600 60  0000 C CNN
-	1    5000 2600
-	1    0    0    -1
-$EndComp
-Wire Wire Line
-	5000 2200 5000 2500
-Wire Wire Line
-	5000 2500 5000 2600
-Text HLabel 4050 2000 0    60   Input ~ 0
+P 5000 3050
+F 0 "#PWR?" H 5000 2800 50  0001 C CNN
+F 1 "GND" H 5000 2900 50  0000 C CNN
+F 2 "" H 5000 3050 60  0000 C CNN
+F 3 "" H 5000 3050 60  0000 C CNN
+	1    5000 3050
+	1    0    0    -1
+$EndComp
+Text HLabel 3750 2000 0    60   Input ~ 0
 Vin
 Wire Wire Line
-	4050 2000 4250 2000
+	3750 2000 4250 2000
 Wire Wire Line
 	4250 2000 4700 2000
@@
 	5300 2000 5650 2000
 Wire Wire Line
-	5650 2000 5850 2000
+	5650 2000 6350 2000
 $Comp
 L CONN_01X01 P?
@@
 Wire Wire Line
 	5650 1800 5650 2000
+Wire Wire Line
+	5650 2000 5650 2150
 Connection ~ 5650 2000
+Wire Wire Line
+	5500 4000 6350 4000
+Wire Wire Line
+	6350 4000 6600 4000
+$Comp
+L C C?
+U 1 1 5565DDF6
+P 6350 4350
+F 0 "C?" H 6375 4450 50  0000 L CNN
+F 1 "1u" H 6375 4250 50  0000 L CNN
+F 2 "" H 6388 4200 30  0000 C CNN
+F 3 "" H 6350 4350 60  0000 C CNN
+	1    6350 4350
+	1    0    0    -1
+$EndComp
+Wire Wire Line
+	6350 3850 6350 4000
+Wire Wire Line
+	6350 4000 6350 4200
+Connection ~ 6350 4000
+Wire Wire Line
+	6350 4500 6350 4800
+$Comp
+L GND #PWR?
+U 1 1 5565DE90
+P 6350 4800
+F 0 "#PWR?" H 6350 4550 50  0001 C CNN
+F 1 "GND" H 6350 4650 50  0000 C CNN
+F 2 "" H 6350 4800 60  0000 C CNN
+F 3 "" H 6350 4800 60  0000 C CNN
+	1    6350 4800
+	1    0    0    -1
+$EndComp
+Text HLabel 6350 2000 2    60   Output ~ 0
+Vcc
+Text HLabel 6600 4000 2    60   Output ~ 0
+Vbb
+Text HLabel 3500 4000 0    60   Input ~ 0
+Vin
+Wire Wire Line
+	4250 1800 4250 2000
+Wire Wire Line
+	4250 2000 4250 2150
+$Comp
+L CONN_01X01 P?
+U 1 1 5565EA50
+P 3700 2950
+F 0 "P?" H 3700 3050 50  0000 C CNN
+F 1 "GND" H 3700 2850 50  0000 C CNN
+F 2 "" H 3700 2950 60  0000 C CNN
+F 3 "" H 3700 2950 60  0000 C CNN
+	1    3700 2950
+	-1   0    0    1
+$EndComp
+Wire Wire Line
+	3900 2950 4250 2950
+Wire Wire Line
+	4250 2950 5000 2950
+Wire Wire Line
+	5000 2950 5650 2950
+Connection ~ 5000 2950
+$Comp
+L CONN_01X01 P?
+U 1 1 5565EC08
+P 6350 3650
+F 0 "P?" V 6350 3500 50  0000 C CNN
+F 1 "Vbb" V 6450 3650 50  0000 C CNN
+F 2 "" H 6350 3650 60  0000 C CNN
+F 3 "" H 6350 3650 60  0000 C CNN
+	1    6350 3650
+	0    -1   -1   0
+$EndComp
+$Comp
+L GND #PWR?
+U 1 1 556C9868
+P 5050 4800
+F 0 "#PWR?" H 5050 4550 50  0001 C CNN
+F 1 "GND" H 5050 4650 50  0000 C CNN
+F 2 "" H 5050 4800 60  0000 C CNN
+F 3 "" H 5050 4800 60  0000 C CNN
+	1    5050 4800
+	1    0    0    -1
+$EndComp
+$Comp
+L R R?
+U 1 1 556C98C6
+P 4300 4250
+F 0 "R?" V 4380 4250 50  0000 C CNN
+F 1 "0" V 4300 4250 50  0000 C CNN
+F 2 "" V 4230 4250 30  0000 C CNN
+F 3 "" H 4300 4250 30  0000 C CNN
+	1    4300 4250
+	1    0    0    -1
+$EndComp
 $Comp
 L LD2979 U?
-U 1 1 5565DC6E
-P 5050 3450
-F 0 "U?" H 5250 3000 50  0000 C CNN
-F 1 "LD2979" H 5050 3600 50  0000 C CNN
-F 2 "" H 5050 3450 60  0000 C CNN
-F 3 "" H 5050 3450 60  0000 C CNN
-	1    5050 3450
-	1    0    0    -1
-$EndComp
-Wire Wire Line
-	4000 3450 4250 3450
-Wire Wire Line
-	4250 3450 4750 3450
+U 1 1 556C9A30
+P 5050 4000
+F 0 "U?" H 5350 3350 50  0000 C CNN
+F 1 "LD2979" H 5050 4150 50  0000 C CNN
+F 2 "" H 5050 4000 60  0000 C CNN
+F 3 "" H 5050 4000 60  0000 C CNN
+	1    5050 4000
+	1    0    0    -1
+$EndComp
+Wire Wire Line
+	5050 4700 5050 4800
+Wire Wire Line
+	3500 4000 3750 4000
+Wire Wire Line
+	3750 4000 4300 4000
+Wire Wire Line
+	4300 4000 4600 4000
+Wire Wire Line
+	4300 4000 4300 4100
+Connection ~ 4300 4000
+Wire Wire Line
+	4300 4400 4300 4500
+Wire Wire Line
+	4300 4500 4600 4500
+$Comp
+L C C?
+U 1 1 556C9E21
+P 4250 2300
+F 0 "C?" H 4275 2400 50  0000 L CNN
+F 1 "1u" H 4275 2200 50  0000 L CNN
+F 2 "" H 4288 2150 30  0000 C CNN
+F 3 "" H 4250 2300 60  0000 C CNN
+F 4 "Value" H 4250 2300 60  0001 C CNN "MPN"
+F 5 "Value" H 4250 2300 60  0001 C CNN "ConradPN"
+	1    4250 2300
+	1    0    0    -1
+$EndComp
+$Comp
+L C C?
+U 1 1 556C9E5C
+P 5650 2300
+F 0 "C?" H 5675 2400 50  0000 L CNN
+F 1 "1u" H 5675 2200 50  0000 L CNN
+F 2 "" H 5688 2150 30  0000 C CNN
+F 3 "" H 5650 2300 60  0000 C CNN
+	1    5650 2300
+	1    0    0    -1
+$EndComp
+Wire Wire Line
+	5000 2200 5000 2950
+Wire Wire Line
+	5000 2950 5000 3050
+Wire Wire Line
+	4250 2450 4250 2950
+Connection ~ 4250 2950
+Wire Wire Line
+	5650 2950 5650 2450
+Connection ~ 3750 4000
+Wire Wire Line
+	3750 4000 3750 4200
 $Comp
 L C C?
 U 1 1 5565DCBC
-P 4250 3800
-F 0 "C?" H 4275 3900 50  0000 L CNN
-F 1 "100n" H 4275 3700 50  0000 L CNN
-F 2 "" H 4288 3650 30  0000 C CNN
-F 3 "" H 4250 3800 60  0000 C CNN
-	1    4250 3800
-	1    0    0    -1
-$EndComp
-$Comp
-L R R?
-U 1 1 5565DCEF
-P 4650 4150
-F 0 "R?" V 4730 4150 50  0000 C CNN
-F 1 "0" V 4650 4150 50  0000 C CNN
-F 2 "" V 4580 4150 30  0000 C CNN
-F 3 "" H 4650 4150 30  0000 C CNN
-	1    4650 4150
-	1    0    0    -1
-$EndComp
-Connection ~ 4250 3450
+P 3750 4350
+F 0 "C?" H 3775 4450 50  0000 L CNN
+F 1 "1u" H 3775 4250 50  0000 L CNN
+F 2 "" H 3788 4200 30  0000 C CNN
+F 3 "" H 3750 4350 60  0000 C CNN
+	1    3750 4350
+	1    0    0    -1
+$EndComp
 $Comp
 L GND #PWR?
 U 1 1 5565DD5B
-P 4250 4600
-F 0 "#PWR?" H 4250 4350 50  0001 C CNN
-F 1 "GND" H 4250 4450 50  0000 C CNN
-F 2 "" H 4250 4600 60  0000 C CNN
-F 3 "" H 4250 4600 60  0000 C CNN
-	1    4250 4600
-	1    0    0    -1
-$EndComp
-Wire Wire Line
-	4250 3950 4250 4500
-Wire Wire Line
-	4250 4500 4250 4600
-Wire Wire Line
-	4750 3700 4650 3700
-Wire Wire Line
-	4650 3700 4650 4000
-Wire Wire Line
-	4650 4300 4650 4500
-Wire Wire Line
-	4650 4500 4250 4500
-Connection ~ 4250 4500
-Wire Wire Line
-	5350 3450 5650 3450
-Wire Wire Line
-	5650 3450 5900 3450
-$Comp
-L C C?
-U 1 1 5565DDF6
-P 5650 3800
-F 0 "C?" H 5675 3900 50  0000 L CNN
-F 1 "4.7u" H 5675 3700 50  0000 L CNN
-F 2 "" H 5688 3650 30  0000 C CNN
-F 3 "" H 5650 3800 60  0000 C CNN
-	1    5650 3800
-	1    0    0    -1
-$EndComp
-Wire Wire Line
-	5650 3300 5650 3450
-Wire Wire Line
-	5650 3450 5650 3650
-Connection ~ 5650 3450
-$Comp
-L R R?
-U 1 1 5565DE49
-P 5650 4300
-F 0 "R?" V 5730 4300 50  0000 C CNN
-F 1 "3.3" V 5650 4300 50  0000 C CNN
-F 2 "" V 5580 4300 30  0000 C CNN
-F 3 "" H 5650 4300 30  0000 C CNN
-	1    5650 4300
-	1    0    0    -1
-$EndComp
-Wire Wire Line
-	5650 3950 5650 4150
-$Comp
-L GND #PWR?
-U 1 1 5565DE90
-P 5650 4600
-F 0 "#PWR?" H 5650 4350 50  0001 C CNN
-F 1 "GND" H 5650 4450 50  0000 C CNN
-F 2 "" H 5650 4600 60  0000 C CNN
-F 3 "" H 5650 4600 60  0000 C CNN
-	1    5650 4600
-	1    0    0    -1
-$EndComp
-Wire Wire Line
-	5650 4450 5650 4600
-Text HLabel 5850 2000 2    60   Output ~ 0
-Vcc
-Text HLabel 5900 3450 2    60   Output ~ 0
-Vbb
-Wire Wire Line
-	4250 3450 4250 3650
-Text HLabel 4000 3450 0    60   Input ~ 0
-Vin
-Wire Wire Line
-	4250 1800 4250 2000
-$Comp
-L CONN_01X01 P?
-U 1 1 5565EA50
-P 4100 2500
-F 0 "P?" H 4100 2600 50  0000 C CNN
-F 1 "GND" H 4100 2400 50  0000 C CNN
-F 2 "" H 4100 2500 60  0000 C CNN
-F 3 "" H 4100 2500 60  0000 C CNN
-	1    4100 2500
-	-1   0    0    1
-$EndComp
-Wire Wire Line
-	4300 2500 5000 2500
-Connection ~ 5000 2500
-$Comp
-L CONN_01X01 P?
-U 1 1 5565EC08
-P 5650 3100
-F 0 "P?" V 5650 2950 50  0000 C CNN
-F 1 "Vbb" V 5750 3100 50  0000 C CNN
-F 2 "" H 5650 3100 60  0000 C CNN
-F 3 "" H 5650 3100 60  0000 C CNN
-	1    5650 3100
-	0    -1   -1   0
-$EndComp
+P 3750 4800
+F 0 "#PWR?" H 3750 4550 50  0001 C CNN
+F 1 "GND" H 3750 4650 50  0000 C CNN
+F 2 "" H 3750 4800 60  0000 C CNN
+F 3 "" H 3750 4800 60  0000 C CNN
+	1    3750 4800
+	1    0    0    -1
+$EndComp
+Wire Wire Line
+	3750 4500 3750 4800
 $EndSCHEMATC

Commit message: Generated the Netlist and started associating footprints
Parts:
- C201, C202, C203, C204: renamed from C?; footprint (none) -> Capacitors_SMD:C_0805_HandSoldering
- P201, P202, P203, P204: renamed from P?; footprint (none) -> Pin_Headers:Pin_Header_Straight_1x01
- R201: renamed from R?; footprint (none) -> Resistors_SMD:R_0805_HandSoldering
- U201: renamed from U?; footprint (none) -> tfac-footprints:SOT-23A
- U202: renamed from U?; footprint (none) -> tfac-footprints:SOT-23-5L
Connections:
- wire segments 29 -> 18
Changed lines of the file:
@@
 LIBS:valves
 LIBS:Tfac-Symbols
+LIBS:TfaC-cache
 EELAYER 25 0
 EELAYER END
@@
 $EndDescr
 $Comp
-L MCP1703T-5002E/CB U?
+L MCP1703T-5002E/CB U201
 U 1 1 5565D3BF
 P 5000 2000
-F 0 "U?" H 5100 1850 50  0000 C CNN
+F 0 "U201" H 5100 1850 50  0000 C CNN
 F 1 "MCP1703T-5002E/CB" H 5000 2150 50  0000 C CNN
-F 2 "" H 5000 2000 60  0000 C CNN
+F 2 "tfac-footprints:SOT-23A" H 5000 2000 60  0001 C CNN
 F 3 "http://ww1.microchip.com/downloads/en/DeviceDoc/22049e.pdf" H 5000 2000 60  0001 C CNN
 F 4 "MCP1703T-5002E/CB" H 5000 2000 60  0001 C CNN "MPN"
@@
 $EndComp
 $Comp
-L GND #PWR?
+L GND #PWR02
 U 1 1 5565D42B
 P 5000 3050
-F 0 "#PWR?" H 5000 2800 50  0001 C CNN
+F 0 "#PWR02" H 5000 2800 50  0001 C CNN
 F 1 "GND" H 5000 2900 50  0000 C CNN
 F 2 "" H 5000 3050 60  0000 C CNN
@@
 Vin
 Wire Wire Line
-	3750 2000 4250 2000
-Wire Wire Line
-	4250 2000 4700 2000
-$Comp
-L CONN_01X01 P?
+	3750 2000 4700 2000
+$Comp
+L CONN_01X01 P202
 U 1 1 5565D452
 P 4250 1600
-F 0 "P?" V 4250 1450 50  0000 C CNN
+F 0 "P202" V 4250 1450 50  0000 C CNN
 F 1 "Vin" V 4350 1600 50  0000 C CNN
-F 2 "" H 4250 1600 60  0000 C CNN
+F 2 "Pin_Headers:Pin_Header_Straight_1x01" H 4250 1600 60  0001 C CNN
 F 3 "" H 4250 1600 60  0000 C CNN
 	1    4250 1600
@@
 Connection ~ 4250 2000
 Wire Wire Line
-	5300 2000 5650 2000
-Wire Wire Line
-	5650 2000 6350 2000
-$Comp
-L CONN_01X01 P?
+	5300 2000 6350 2000
+$Comp
+L CONN_01X01 P203
 U 1 1 5565D4A7
 P 5650 1600
-F 0 "P?" V 5650 1500 50  0000 C CNN
+F 0 "P203" V 5650 1500 50  0000 C CNN
 F 1 "Vcc" V 5750 1600 50  0000 C CNN
-F 2 "" H 5650 1600 60  0000 C CNN
+F 2 "Pin_Headers:Pin_Header_Straight_1x01" H 5650 1600 60  0001 C CNN
 F 3 "" H 5650 1600 60  0000 C CNN
 	1    5650 1600
@@
 $EndComp
 Wire Wire Line
-	5650 1800 5650 2000
-Wire Wire Line
-	5650 2000 5650 2150
+	5650 1800 5650 2150
 Connection ~ 5650 2000
 Wire Wire Line
-	5500 4000 6350 4000
-Wire Wire Line
-	6350 4000 6600 4000
-$Comp
-L C C?
+	5500 4000 6600 4000
+$Comp
+L C C204
 U 1 1 5565DDF6
 P 6350 4350
-F 0 "C?" H 6375 4450 50  0000 L CNN
+F 0 "C204" H 6375 4450 50  0000 L CNN
 F 1 "1u" H 6375 4250 50  0000 L CNN
-F 2 "" H 6388 4200 30  0000 C CNN
+F 2 "Capacitors_SMD:C_0805_HandSoldering" H 6388 4200 30  0001 C CNN
 F 3 "" H 6350 4350 60  0000 C CNN
 	1    6350 4350
@@
 $EndComp
 Wire Wire Line
-	6350 3850 6350 4000
-Wire Wire Line
-	6350 4000 6350 4200
+	6350 3850 6350 4200
 Connection ~ 6350 4000
 Wire Wire Line
 	6350 4500 6350 4800
 $Comp
-L GND #PWR?
+L GND #PWR03
 U 1 1 5565DE90
 P 6350 4800
-F 0 "#PWR?" H 6350 4550 50  0001 C CNN
+F 0 "#PWR03" H 6350 4550 50  0001 C CNN
 F 1 "GND" H 6350 4650 50  0000 C CNN
 F 2 "" H 6350 4800 60  0000 C CNN
@@
 Vin
 Wire Wire Line
-	4250 1800 4250 2000
-Wire Wire Line
-	4250 2000 4250 2150
-$Comp
-L CONN_01X01 P?
+	4250 1800 4250 2150
+$Comp
+L CONN_01X01 P201
 U 1 1 5565EA50
 P 3700 2950
-F 0 "P?" H 3700 3050 50  0000 C CNN
+F 0 "P201" H 3700 3050 50  0000 C CNN
 F 1 "GND" H 3700 2850 50  0000 C CNN
-F 2 "" H 3700 2950 60  0000 C CNN
+F 2 "Pin_Headers:Pin_Header_Straight_1x01" H 3700 2950 60  0001 C CNN
 F 3 "" H 3700 2950 60  0000 C CNN
 	1    3700 2950
@@
 $EndComp
 Wire Wire Line
-	3900 2950 4250 2950
-Wire Wire Line
-	4250 2950 5000 2950
-Wire Wire Line
-	5000 2950 5650 2950
+	3900 2950 5650 2950
 Connection ~ 5000 2950
 $Comp
-L CONN_01X01 P?
+L CONN_01X01 P204
 U 1 1 5565EC08
 P 6350 3650
-F 0 "P?" V 6350 3500 50  0000 C CNN
+F 0 "P204" V 6350 3500 50  0000 C CNN
 F 1 "Vbb" V 6450 3650 50  0000 C CNN
-F 2 "" H 6350 3650 60  0000 C CNN
+F 2 "Pin_Headers:Pin_Header_Straight_1x01" H 6350 3650 60  0001 C CNN
 F 3 "" H 6350 3650 60  0000 C CNN
 	1    6350 3650
@@
 $EndComp
 $Comp
-L GND #PWR?
+L GND #PWR04
 U 1 1 556C9868
 P 5050 4800
-F 0 "#PWR?" H 5050 4550 50  0001 C CNN
+F 0 "#PWR04" H 5050 4550 50  0001 C CNN
 F 1 "GND" H 5050 4650 50  0000 C CNN
 F 2 "" H 5050 4800 60  0000 C CNN
@@
 $EndComp
 $Comp
-L R R?
+L R R201
 U 1 1 556C98C6
 P 4300 4250
-F 0 "R?" V 4380 4250 50  0000 C CNN
+F 0 "R201" V 4380 4250 50  0000 C CNN
 F 1 "0" V 4300 4250 50  0000 C CNN
-F 2 "" V 4230 4250 30  0000 C CNN
+F 2 "Resistors_SMD:R_0805_HandSoldering" V 4230 4250 30  0001 C CNN
 F 3 "" H 4300 4250 30  0000 C CNN
 	1    4300 4250
@@
 $EndComp
 $Comp
-L LD2979 U?
+L LD2979 U202
 U 1 1 556C9A30
 P 5050 4000
-F 0 "U?" H 5350 3350 50  0000 C CNN
+F 0 "U202" H 5350 3350 50  0000 C CNN
 F 1 "LD2979" H 5050 4150 50  0000 C CNN
-F 2 "" H 5050 4000 60  0000 C CNN
+F 2 "tfac-footprints:SOT-23-5L" H 5050 4000 60  0001 C CNN
 F 3 "" H 5050 4000 60  0000 C CNN
 	1    5050 4000
@@
 	5050 4700 5050 4800
 Wire Wire Line
-	3500 4000 3750 4000
-Wire Wire Line
-	3750 4000 4300 4000
-Wire Wire Line
-	4300 4000 4600 4000
+	3500 4000 4600 4000
 Wire Wire Line
 	4300 4000 4300 4100
@@
 	4300 4500 4600 4500
 $Comp
-L C C?
+L C C202
 U 1 1 556C9E21
 P 4250 2300
-F 0 "C?" H 4275 2400 50  0000 L CNN
+F 0 "C202" H 4275 2400 50  0000 L CNN
 F 1 "1u" H 4275 2200 50  0000 L CNN
-F 2 "" H 4288 2150 30  0000 C CNN
+F 2 "Capacitors_SMD:C_0805_HandSoldering" H 4288 2150 30  0001 C CNN
 F 3 "" H 4250 2300 60  0000 C CNN
 F 4 "Value" H 4250 2300 60  0001 C CNN "MPN"
@@
 $EndComp
 $Comp
-L C C?
+L C C203
 U 1 1 556C9E5C
 P 5650 2300
-F 0 "C?" H 5675 2400 50  0000 L CNN
+F 0 "C203" H 5675 2400 50  0000 L CNN
 F 1 "1u" H 5675 2200 50  0000 L CNN
-F 2 "" H 5688 2150 30  0000 C CNN
+F 2 "Capacitors_SMD:C_0805_HandSoldering" H 5688 2150 30  0001 C CNN
 F 3 "" H 5650 2300 60  0000 C CNN
 	1    5650 2300
@@
 $EndComp
 Wire Wire Line
-	5000 2200 5000 2950
-Wire Wire Line
-	5000 2950 5000 3050
+	5000 2200 5000 3050
 Wire Wire Line
 	4250 2450 4250 2950
@@
 	3750 4000 3750 4200
 $Comp
-L C C?
+L C C201
 U 1 1 5565DCBC
 P 3750 4350
-F 0 "C?" H 3775 4450 50  0000 L CNN
+F 0 "C201" H 3775 4450 50  0000 L CNN
 F 1 "1u" H 3775 4250 50  0000 L CNN
-F 2 "" H 3788 4200 30  0000 C CNN
+F 2 "Capacitors_SMD:C_0805_HandSoldering" H 3788 4200 30  0001 C CNN
 F 3 "" H 3750 4350 60  0000 C CNN
 	1    3750 4350
@@
 $EndComp
 $Comp
-L GND #PWR?
+L GND #PWR05
 U 1 1 5565DD5B
 P 3750 4800
-F 0 "#PWR?" H 3750 4550 50  0001 C CNN
+F 0 "#PWR05" H 3750 4550 50  0001 C CNN
 F 1 "GND" H 3750 4650 50  0000 C CNN
 F 2 "" H 3750 4800 60  0000 C CNN

Commit message: Started the layout
Parts:
- removed P201: GND, Pin_Headers:Pin_Header_Straight_1x01, symbol CONN_01X01
- removed P202: Vin, Pin_Headers:Pin_Header_Straight_1x01, symbol CONN_01X01
- removed P203: Vcc, Pin_Headers:Pin_Header_Straight_1x01, symbol CONN_01X01
- removed P204: Vbb, Pin_Headers:Pin_Header_Straight_1x01, symbol CONN_01X01
Changed lines of the file:
@@
 Wire Wire Line
 	3750 2000 4700 2000
-$Comp
-L CONN_01X01 P202
-U 1 1 5565D452
-P 4250 1600
-F 0 "P202" V 4250 1450 50  0000 C CNN
-F 1 "Vin" V 4350 1600 50  0000 C CNN
-F 2 "Pin_Headers:Pin_Header_Straight_1x01" H 4250 1600 60  0001 C CNN
-F 3 "" H 4250 1600 60  0000 C CNN
-	1    4250 1600
-	0    -1   -1   0
-$EndComp
-Connection ~ 4250 2000
 Wire Wire Line
 	5300 2000 6350 2000
-$Comp
-L CONN_01X01 P203
-U 1 1 5565D4A7
-P 5650 1600
-F 0 "P203" V 5650 1400 50  0000 C CNN
-F 1 "Vcc" V 5750 1600 50  0000 C CNN
-F 2 "Pin_Headers:Pin_Header_Straight_1x01" H 5650 1600 60  0001 C CNN
-F 3 "" H 5650 1600 60  0000 C CNN
-	1    5650 1600
-	0    -1   -1   0
-$EndComp
-Wire Wire Line
-	5650 1800 5650 2150
-Connection ~ 5650 2000
 Wire Wire Line
 	5500 4000 6600 4000
@@
 	1    0    0    -1
 $EndComp
-Wire Wire Line
-	6350 3850 6350 4200
-Connection ~ 6350 4000
 Wire Wire Line
 	6350 4500 6350 4800
@@
 Text HLabel 3500 4000 0    60   Input ~ 0
 Vin
-Wire Wire Line
-	4250 1800 4250 2150
-$Comp
-L CONN_01X01 P201
-U 1 1 5565EA50
-P 3700 2950
-F 0 "P201" H 3700 3050 50  0000 C CNN
-F 1 "GND" H 3700 2850 50  0000 C CNN
-F 2 "Pin_Headers:Pin_Header_Straight_1x01" H 3700 2950 60  0001 C CNN
-F 3 "" H 3700 2950 60  0000 C CNN
-	1    3700 2950
-	-1   0    0    1
-$EndComp
-Wire Wire Line
-	3900 2950 5650 2950
 Connection ~ 5000 2950
-$Comp
-L CONN_01X01 P204
-U 1 1 5565EC08
-P 6350 3650
-F 0 "P204" V 6350 3500 50  0000 C CNN
-F 1 "Vbb" V 6450 3650 50  0000 C CNN
-F 2 "Pin_Headers:Pin_Header_Straight_1x01" H 6350 3650 60  0001 C CNN
-F 3 "" H 6350 3650 60  0000 C CNN
-	1    6350 3650
-	0    -1   -1   0
-$EndComp
 $Comp
 L GND #PWR04
@@
 U 1 1 556C9A30
 P 5050 4000
+AR Path="/556C9A30" Ref="U202"  Part="1"
+AR Path="/5560D23E/556C9A30" Ref="U202"  Part="1"
 F 0 "U202" H 5350 3350 50  0000 C CNN
 F 1 "LD2979" H 5050 4150 50  0000 C CNN
@@
 Wire Wire Line
 	4250 2450 4250 2950
-Connection ~ 4250 2950
 Wire Wire Line
 	5650 2950 5650 2450
@@
 Wire Wire Line
 	3750 4500 3750 4800
+Wire Wire Line
+	4250 2150 4250 2000
+Connection ~ 4250 2000
+Wire Wire Line
+	5650 2150 5650 2000
+Connection ~ 5650 2000
+Wire Wire Line
+	6350 4200 6350 4000
+Connection ~ 6350 4000
+Wire Wire Line
+	4250 2950 5650 2950
 $EndSCHEMATC

Commit message: Getting up to date
Parts:
- U202: symbol LD2979 -> LD2979-RESCUE-TfaC
Changed lines of the file:
@@
 EESchema Schematic File Version 2
+LIBS:TfaC-rescue
 LIBS:power
 LIBS:device
@@
 $EndComp
 $Comp
-L LD2979 U202
+L LD2979-RESCUE-TfaC U202
 U 1 1 556C9A30
 P 5050 4000
