File: PCB/powerSystem.sch (KiCad schematic (older format))
At the start: 11 parts, among them U201 MCP1703T-5002E/CB, U202 LD2979

Commit message: Added alarm
Parts:
- added W? (x2): TEST_1P, symbol TEST_1P
Connections:
- net Vbb: now also W?.1
- net Vcc: now also W?.1
Changed lines of the file:
@@
 	7300 5300 7300 5550
 Connection ~ 7300 4000
+$Comp
+L TEST_1P W?
+U 1 1 56E53D9F
+P 6900 1500
+F 0 "W?" H 6900 1770 50  0000 C CNN
+F 1 "TEST_1P" H 6900 1700 50  0000 C CNN
+F 2 "" H 7100 1500 50  0000 C CNN
+F 3 "" H 7100 1500 50  0000 C CNN
+	1    6900 1500
+	1    0    0    -1
+$EndComp
+Wire Wire Line
+	6900 1500 6900 1600
+Connection ~ 6900 1600
+$Comp
+L TEST_1P W?
+U 1 1 56E53EC3
+P 7500 3950
+F 0 "W?" H 7500 4220 50  0000 C CNN
+F 1 "TEST_1P" H 7500 4150 50  0000 C CNN
+F 2 "" H 7700 3950 50  0000 C CNN
+F 3 "" H 7700 3950 50  0000 C CNN
+	1    7500 3950
+	1    0    0    -1
+$EndComp
+Wire Wire Line
+	7500 3950 7500 4000
+Connection ~ 7500 4000
 $EndSCHEMATC

Commit message: Re-organised the board to incorporate the MISO
Parts:
- D201, D202: footprint LEDs:LED-0805 -> LEDs:LED_0805
- W201, W202: renamed from W?; footprint (none) -> Measurement_Points:Measurement_Point_Round-SMD-Pad_Small
Changed lines of the file:
@@
 F 0 "D201" H 6700 2100 50  0000 C CNN
 F 1 "LED" H 6700 1900 50  0000 C CNN
-F 2 "LEDs:LED-0805" H 6700 2000 60  0001 C CNN
+F 2 "LEDs:LED_0805" H 6700 2000 60  0001 C CNN
 F 3 "" H 6700 2000 60  0000 C CNN
 	1    6700 2000
@@
 F 0 "D202" H 7300 4700 50  0000 C CNN
 F 1 "LED" H 7300 4500 50  0000 C CNN
-F 2 "LEDs:LED-0805" H 7300 4600 60  0001 C CNN
+F 2 "LEDs:LED_0805" H 7300 4600 60  0001 C CNN
 F 3 "" H 7300 4600 60  0000 C CNN
 	1    7300 4600
@@
 Connection ~ 7300 4000
 $Comp
-L TEST_1P W?
+L TEST_1P W201
 U 1 1 56E53D9F
 P 6900 1500
-F 0 "W?" H 6900 1770 50  0000 C CNN
+F 0 "W201" H 6900 1770 50  0000 C CNN
 F 1 "TEST_1P" H 6900 1700 50  0000 C CNN
-F 2 "" H 7100 1500 50  0000 C CNN
+F 2 "Measurement_Points:Measurement_Point_Round-SMD-Pad_Small" H 7100 1500 50  0001 C CNN
 F 3 "" H 7100 1500 50  0000 C CNN
 	1    6900 1500
@@
 Connection ~ 6900 1600
 $Comp
-L TEST_1P W?
+L TEST_1P W202
 U 1 1 56E53EC3
 P 7500 3950
-F 0 "W?" H 7500 4220 50  0000 C CNN
+F 0 "W202" H 7500 4220 50  0000 C CNN
 F 1 "TEST_1P" H 7500 4150 50  0000 C CNN
-F 2 "" H 7700 3950 50  0000 C CNN
+F 2 "Measurement_Points:Measurement_Point_Round-SMD-Pad_Small" H 7700 3950 50  0001 C CNN
 F 3 "" H 7700 3950 50  0000 C CNN
 	1    7500 3950
